File: P2/PCB/Autosense-combined.brd (EAGLE design)
At the start: 89.8 x 41.9 mm, 69 parts, among them IC1 MC1458, IC2 MC1458, IC3 MC1458, IC4 MC1458, K1 G6H2-100, K2 G6H2-100, K3 G6H2-100, K4 G6H2-100, K5 G6H2-100

Commit message: Added ipod-female-breakout
Parts:
- IC1, IC2, IC3, IC4: value MC1458 -> LM358D; device burr-brown:SO08 -> linear:SO08
- K1, K2, K3, K4, K5: value G6H2-100 -> G6K-2G-Y; device relay:G6H2-100 -> relay:G6K-2G-Y
- moved K4 1.94 mm to (35.6, 25.9)
- moved K3 1.94 mm to (50.8, 25.9)
- moved K2 1.81 mm to (66.2, 25.9)
- moved D1-4 1.66 mm to (35.6, 19.2), flipped to the top, turned to 180 degrees
- moved D1-3 1.66 mm to (50.8, 19.2), flipped to the top, turned to 180 degrees
- moved D1-2 1.51 mm to (66.2, 19.2), flipped to the top, turned to 180 degrees
- moved K5 1.11 mm to (20.3, 25.9)
- moved K1 0.97 mm to (79.9, 25.7)
- moved D1-1 0.65 mm to (79.9, 19.1), flipped to the top, turned to 180 degrees
- moved D1-5 0.48 mm to (20.3, 19.2), flipped to the top, turned to 180 degrees
- moved IC4 0.16 mm to (34.1, 8.26)
Connections:
- net $NET1: now also K2.3; no longer K2.P1
- net $NET13: now also K1.3; no longer K1.P1
- net $NET2: now also K3.3; no longer K3.P1
- net $NET3: now also K4.3; no longer K4.P1
- net $NET4: now also K5.3; no longer K5.P1
- net N$1: now also K1.6; no longer K1.P2
- net N$19: now also K2.6; no longer K2.P2
- net N$21: now also K3.6; no longer K3.P2
- net N$28: now also K4.6; no longer K4.P2
- net N$29: now also K5.6; no longer K5.P2
- net OUT0: now also K1.8; no longer K1.10
- net OUT1: now also K2.8; no longer K2.10
- net OUT1-2: now also K1.5, K2.5, K3.5, K4.5, K5.5; no longer K1.S2, K2.S2, K3.S2, K4.S2, K5.S2
- net OUT1-3: now also K1.4, K2.4, K3.4, K4.4, K5.4; no longer K1.S1, K2.S1, K3.S1, K4.S1, K5.S1
- net OUT2: now also K3.8; no longer K3.10
- net OUT3: now also K4.8; no longer K4.10
- net OUT4: now also K5.8; no longer K5.10
Routing:
- net OUT1-3: track 121.3 -> 99.9 mm, vias 4 -> 5
- net OUT1-2: track 140.6 -> 130.1 mm, vias 4 -> 0
- net OUT2: track 68.1 -> 73.3 mm, vias 0 -> 2
- net OUT3: track 22.6 -> 27.5 mm, vias 0 -> 2
- net 5V: track 246.6 -> 251.5 mm, vias 4 -> 9
- net N$19: track 26.6 -> 31.5 mm
- net N$29: track 16.2 -> 11.6 mm
- net $NET3: track 19.7 -> 15.6 mm
- net N$21: track 26.5 -> 30.4 mm
- net $NET2: track 19.3 -> 15.4 mm
- net $NET4: track 15.7 -> 11.9 mm
- net N$28: track 26.9 -> 30.3 mm
- net $NET1: track 19.4 -> 16.2 mm
- net OUT0: track 104.4 -> 107.1 mm, vias 0 -> 2
- net $NET13: track 19.5 -> 17.2 mm
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