File: P2/PCB/Autosense-combined.sch (EAGLE design)
At the start: 24 parts, among them IC1 MC1458, K1 G6H2-100

Commit message: xwoofer crossover with 24db/octave and star ground
xwoofer routed, design rules passed, not pretty
Parts:
- removed C2A, C2B, C5: 100n, rcl:C-EUC0805
- removed C4, C6: 2n, rcl:C-EUC0805
- removed R1A, R3: 10k, resistor:R-EU_R0805
- removed R1B: 10k, rcl:R-EU_M0805
- removed R7, R8: 15k, resistor:R-EU_R0805
- added C3-1, C3-2, CA-1, CA-2, CB-1, CB-2: 100n, rcl:C-EUC0805
- added C4-1, C4-2, C5-1, C5-2: 2n, rcl:C-EUC0805
- added D1-2: (no value), diode:DIODE-GF1
- added IC2: MC1458, burr-brown:OPA2130U
- added K2: G6H2-100, relay:G6H2-100
- added R3-1, R3-2, RA-1, RA-2: 10k, resistor:R-EU_R0805
- added R7-1, R7-2, R8-1, R8-2: 5k, resistor:R-EU_R0805
- added RB-1, RB-2: 10k, rcl:R-EU_M0805
- R1: device rcl:R-EU_R0805 -> rcl:R-EU_R1206
- renumbered D1 to D1-1
Connections:
- removed net J1: D1-1.A, K11.2
- removed net J2: C4.1, IC1B.-IN, IC1B.OUT
- removed net N$15: K13.S, OUT1-1.KL
- removed net N$16: K12.S, OUT1-3.KL
- removed net N$3: OUT1-2.KL, OUT1-4.KL, R1.2, X1-2.KL
- new net $NET1: CB-2.1, K22.P, X2-1.KL
- new net ADC0: C4-1.1, CON1.9, IC1B.-IN, IC1B.OUT
- new net ADC1: C4-2.1, CON1.7, IC2B.-IN, IC2B.OUT
- new net ADC2: CON1.5
- new net ADC3: CON1.3
- new net AGND: C1.-, C5-1.2, C5-2.2, CON1.12, OUT1-2.KL, OUT1-4.KL, R1.2, R5.1, X1-2.KL, X2-2.KL
- new net N$10: IC2A.-IN, R3-2.1, RA-2.1, RB-2.1
- new net N$12: C5-2.1, IC2B.+IN, R8-2.1
- new net N$14: C4-2.2, R7-2.1, R8-2.2
- new net N$17: CA-2.2, RA-2.2
- new net N$18: CB-2.2, RB-2.2
- new net N$19: CA-2.1, K23.P, X2-3.KL
- new net N$7: IC2A.OUT, R3-2.2, R7-2.2
- new net OUT0: CON1.10, D1-1.A, K11.2
- new net OUT1: CON1.8, D1-2.A, K21.2
- new net OUT1-1: K13.S, K23.S, OUT1-1.KL
- new net OUT1-3: K12.S, K22.S, OUT1-3.KL
- new net OUT2: CON1.6
- new net OUT3: CON1.4
- net $NET13: now also CB-1.1; no longer C2B.1
- net 5V: now also C3-1.1, C3-2.1, D1-2.C, IC2A.V+, K21.1; no longer C5.1
- net GND: now also C3-1.2, C3-2.2, IC2A.V-; no longer C1.-, C5.2, C6.2, R5.1
- net N$1: now also CA-1.1; no longer C2A.1
- net N$11: now also CA-1.2, RA-1.2; no longer C2A.2, R1A.2
- net N$13: now also CB-1.2, RB-1.2; no longer C2B.2, R1B.2
- net N$2: now also C5-1.1, R8-1.1; no longer C6.1, R8.1
- net N$6: now also R3-1.1, RA-1.1, RB-1.1; no longer R1A.1, R1B.1, R3.1
- net N$8: now also C4-1.2, R7-1.1, R8-1.2; no longer C4.2, R7.1, R8.2
- net N$9: now also R3-1.2, R7-1.2; no longer R3.2, R7.2
- net V/2: now also IC2A.+IN
Other:
- moved on the sheet: IC1A, IC1B, R1, X1-1, X1-2, X1-3, X2-1, X2-2, X2-3, X3-1, X3-2, X3-3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

Commit message: Autosense 4+1 channels complete
Parts:
- added C3-3, C3-4, CA-3, CA-4, CB-3, CB-4, CV-1, CV-2, CV-3, CV-4: 100n, rcl:C-EUC0805
- added C4-3, C4-4, C5-3, C5-4: 2n, rcl:C-EUC0805
- added D1-3, D1-4, D1-5: (no value), diode:DIODE-GF1
- added IC3, IC4: MC1458, burr-brown:OPA2130U
- added K3, K4, K5: G6H2-100, relay:G6H2-100
- added R3-3, R3-4, RA-3, RA-4: 10k, resistor:R-EU_R0805
- added R7-3, R7-4, R8-3, R8-4: 5k, resistor:R-EU_R0805
- added RB-3, RB-4: 10k, rcl:R-EU_M0805
Connections:
- removed net OUT1-1: K13.S, K23.S, OUT1-1.KL
- new net $NET2: CB-3.1, K32.P, X3-1.KL
- new net $NET3: CB-4.1, K42.P, X4-1.KL
- new net $NET4: K52.P, X5-1.KL
- new net N$15: C4-3.2, R7-3.1, R8-3.2
- new net N$16: CA-3.2, RA-3.2
- new net N$20: CB-3.2, RB-3.2
- new net N$21: CA-3.1, K33.P, X3-3.KL
- new net N$22: IC4A.OUT, R3-4.2, R7-4.2
- new net N$23: IC4A.-IN, R3-4.1, RA-4.1, RB-4.1
- new net N$24: C5-4.1, IC4B.+IN, R8-4.1
- new net N$25: C4-4.2, R7-4.1, R8-4.2
- new net N$26: CA-4.2, RA-4.2
- new net N$27: CB-4.2, RB-4.2
- new net N$28: CA-4.1, K43.P, X4-3.KL
- new net N$29: K53.P, X5-3.KL
- new net N$3: IC3A.OUT, R3-3.2, R7-3.2
- new net N$4: IC3A.-IN, R3-3.1, RA-3.1, RB-3.1
- new net N$5: C5-3.1, IC3B.+IN, R8-3.1
- new net OUT1-2: K13.S, K23.S, K33.S, K43.S, K53.S, OUT1-1.KL
- new net OUT4: CON1.2, D1-5.A, K51.2
- net 5V: now also C3-3.1, C3-4.1, D1-3.C, D1-4.C, D1-5.C, IC3A.V+, IC4A.V+, K31.1, K41.1, K51.1
- net ADC2: now also C4-3.1, IC3B.-IN, IC3B.OUT
- net ADC3: now also C4-4.1, IC4B.-IN, IC4B.OUT
- net AGND: now also C5-3.2, C5-4.2, X3-2.KL, X4-2.KL, X5-2.KL; no longer C1.-, R5.1
- net GND: now also C1.-, C3-3.2, C3-4.2, CV-1.1, CV-2.1, CV-3.1, CV-4.1, IC3A.V-, IC4A.V-, R5.1
- net OUT1-3: now also K32.S, K42.S, K52.S
- net OUT2: now also D1-3.A, K31.2
- net OUT3: now also D1-4.A, K41.2
- net V/2: now also CV-1.2, CV-2.2, CV-3.2, CV-4.2, IC3A.+IN, IC4A.+IN
Other:
- moved on the sheet: C3-1, C3-2, C4-1, C4-2, C5-1, C5-2, CA-1, CA-2, CB-1, CB-2, D1-1, D1-2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

Commit message: Added ipod-female-breakout
Parts:
- IC1, IC2, IC3, IC4: value MC1458 -> LM358D; device burr-brown:OPA2130U -> linear:LM358D
- K1, K2, K3, K4, K5: value G6H2-100 -> G6K-2G-Y; device relay:G6H2-100 -> relay:G6K-2G-Y
Connections:
- net 5V: now also IC1P.V+, IC2P.V+, IC3P.V+, IC4P.V+, K11.+, K21.+, K31.+, K41.+, K51.+; no longer IC1A.V+, IC2A.V+, IC3A.V+, IC4A.V+, K11.1, K21.1, K31.1, K41.1, K51.1
- net GND: now also IC1P.V-, IC2P.V-, IC3P.V-, IC4P.V-; no longer IC1A.V-, IC2A.V-, IC3A.V-, IC4A.V-
- net OUT0: now also K11.-; no longer K11.2
- net OUT1: now also K21.-; no longer K21.2
- net OUT2: now also K31.-; no longer K31.2
- net OUT3: now also K41.-; no longer K41.2
- net OUT4: now also K51.-; no longer K51.2
Other:
- moved on the sheet: C3-1, C3-2, C3-3, C3-4, K1, K2, K3, K4, K5
